File: Quansheng_UV-K5_PCB_R51-V1.4.kicad_sch (KiCad schematic)
At the start: 515 parts, among them J1 USB_C_Receptacle_USB2.0, J2 Conn_Batt_K5, J4 Conn_Coaxial_K5, J5 SJ1-3525N (3.5mm), J6 Connector_Jack_2.5mm_PJ-204, Q1 2SC4226, Q10 Si2301DS, Q11 2SC3052, Q12 DTC114E, Q13 DTC114E, Q14 UMC4N, Q15 Si2301DS, Q16 DTC114E, Q17 UMC4N, Q18 UMC4N, Q19 UMC4N, Q2 DTA114E, Q20 2SC4226, Q21 UMC4N, Q22 2SC4226, Q23 NP6003, Q24 KRC109S, Q25 DTC114E, Q26 DTC114E, Q27 DTC114E, Q3 DTC114E, Q4 2SC4226, Q5 2SK3078A, Q6 DTC114E, Q7 DTC114E?, Q8 RD02LUS2, Q9 DTC114E, SW1 1, SW10 0, SW11 *, SW12 F, SW13 M A, SW14 UP B, SW15 DOWN C, SW16 EXIT D, SW17 PTT, SW18 I, SW19 II, SW2 2, SW3 3, SW4 4, SW5 5, SW6 6, SW7 7, SW8 8, SW9 9, U1 BEKEN BK4819, U10 KC2520Z, U2 DP32G030, U3 AT24CS64-SSHM, U4 LN4898, U5 XS5822, U6 H3601, U7 BK1080, U8 LM2904, U9 MD53U33

Commit message: First attempts at RF path annotation
Other:
- note added: "DC Path for TX UHF PIN"
- note added: "DC Path for TX VHF PIN"
- note added: "RX PIN Switching"
- note added: "RX mute PIN"
- note added: "RX_EN"
- note added: "RX_UHF_EN"
- note added: "RX_VHF_EN"
- note added: "Regulated UHF PIN TX Bias?"
- note added: "TX driver bias"
- note added: "TX_EN"
- note added: "TX_UHF_EN"
- note added: "TX_VHF_EN"
- note added: "UHF LNA"
- note added: "UHF PIN TX Bias"
- note added: "UHF TX"
- note added: "UHF TX LPF"
- note added: "UHF filter"
- note added: "UHF pre-filter"
- note added: "VHF LNA"
- note added: "VHF TX"
- note added: "VHF TX LPF"
- note added: "VHF filter"
- note added: "VHF/FM/Air pre-filter"
Changed lines of the file:
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@@
+    (effects (font (size 1.27 1.27) (thickness 0.254) bold) (justify left bottom))
+  )
+  (text "RX PIN Switching" (at 582.93 139.7 0)
     (effects (font (size 1.27 1.27) (thickness 0.254) bold) (justify left bottom))
   )
@@
     (effects (font (size 1.27 1.27) (thickness 0.254) bold) (justify left bottom))
   )
+  (text "RX mute PIN" (at 650.24 129.54 0)
+    (effects (font (size 1.27 1.27) (thickness 0.254) bold) (justify left bottom))
+  )
+  (text "VHF TX LPF" (at 495.3 246.38 0)
+    (effects (font (size 1.27 1.27) (thickness 0.254) bold) (justify left bottom))
+  )
   (text "TX LED" (at 538.226 350.012 0)
+    (effects (font (size 1.27 1.27) (thickness 0.254) bold) (justify left bottom))
+  )
+  (text "UHF LNA" (at 626.11 106.68 0)
     (effects (font (size 1.27 1.27) (thickness 0.254) bold) (justify left bottom))
   )
@@
     (effects (font (size 1.27 1.27) (thickness 0.254) bold) (justify left bottom))
   )
+  (text "Regulated UHF PIN TX Bias?" (at 617.22 222.25 0)
+    (effects (font (size 1.27 1.27) (thickness 0.254) bold) (justify left bottom))
+  )
   (text "PA10 Col 1" (at 315.214 434.594 90)
     (effects (font (size 1.27 1.27)) (justify left bottom))
+  )
+  (text "UHF TX LPF" (at 626.11 175.26 0)
+    (effects (font (size 1.27 1.27) (thickness 0.254) bold) (justify left bottom))
   )
   (text "Combined volume pot.\n& ON/OFF Switch\n" (at 244.856 401.066 0)
@@
     (effects (font (size 1.27 1.27) (thickness 0.254) bold) (justify left bottom))
   )
+  (text "DC Path for TX VHF PIN" (at 722.63 207.01 0)
+    (effects (font (size 1.27 1.27) (thickness 0.254) bold) (justify left bottom))
+  )
   (text "Audio amplifier" (at 198.374 346.456 0)
+    (effects (font (size 1.27 1.27) (thickness 0.254) bold) (justify left bottom))
+  )
+  (text "UHF pre-filter" (at 643.89 80.01 0)
     (effects (font (size 1.27 1.27) (thickness 0.254) bold) (justify left bottom))
   )
@@
     (effects (font (size 1.27 1.27)) (justify left bottom))
   )
+  (text "VHF/FM/Air pre-filter" (at 675.64 116.84 0)
+    (effects (font (size 1.27 1.27) (thickness 0.254) bold) (justify left bottom))
+  )
   (text "DAN222-B\ncommon cathode\ninternally connected\nto DAN222-A"
     (at 427.482 376.428 0)
@@
     (effects (font (size 1.27 1.27) (thickness 0.254) bold) (justify left bottom))
   )
+  (text "VHF filter" (at 595.63 43.18 0)
+    (effects (font (size 1.27 1.27) (thickness 0.254) bold) (justify left bottom))
+  )
   (text "Flashlight LED" (at 577.088 350.266 0)
+    (effects (font (size 1.27 1.27) (thickness 0.254) bold) (justify left bottom))
+  )
+  (text "UHF PIN TX Bias" (at 486.41 218.44 0)
+    (effects (font (size 1.27 1.27) (thickness 0.254) bold) (justify left bottom))
+  )
+  (text "UHF filter" (at 584.2 100.33 0)
+    (effects (font (size 1.27 1.27) (thickness 0.254) bold) (justify left bottom))
+  )
+  (text "RX_EN" (at 411.48 130.81 0)
+    (effects (font (size 1.27 1.27) (thickness 0.254) bold) (justify left bottom))
+  )
+  (text "RX_VHF_EN" (at 414.02 59.69 0)
     (effects (font (size 1.27 1.27) (thickness 0.254) bold) (justify left bottom))
   )
@@
     (effects (font (size 1.27 1.27) (thickness 0.254) bold) (justify left bottom))
   )
+  (text "VHF LNA" (at 711.2 85.09 0)
+    (effects (font (size 1.27 1.27) (thickness 0.254) bold) (justify left bottom))
+  )
   (text "USB charge circuit" (at 561.34 470.408 0)
+    (effects (font (size 1.27 1.27) (thickness 0.254) bold) (justify left bottom))
+  )
+  (text "TX_VHF_EN" (at 267.97 292.1 0)
     (effects (font (size 1.27 1.27) (thickness 0.254) bold) (justify left bottom))
   )
@@
     (effects (font (size 1.27 1.27) (thickness 0.254) bold) (justify left bottom))
   )
+  (text "TX_EN" (at 264.16 128.27 0)
+    (effects (font (size 1.27 1.27) (thickness 0.254) bold) (justify left bottom))
+  )
   (text "Battery filtering and current limiting" (at 396.748 520.954 0)
+    (effects (font (size 1.27 1.27) (thickness 0.254) bold) (justify left bottom))
+  )
+  (text "RX_UHF_EN" (at 406.4 101.6 0)
     (effects (font (size 1.27 1.27) (thickness 0.254) bold) (justify left bottom))
   )
@@
     (effects (font (size 1.27 1.27) (thickness 0.254) bold) (justify left bottom))
   )
+  (text "TX_UHF_EN" (at 267.97 243.84 0)
+    (effects (font (size 1.27 1.27) (thickness 0.254) bold) (justify left bottom))
+  )
+  (text "UHF TX" (at 513.08 175.26 0)
+    (effects (font (size 1.27 1.27) (thickness 0.254) bold) (justify left bottom))
+  )
   (text "PA3  Keypad Row 1\nPA4  Keypad Row 2\nPA5  Keypad Row 3\nPA6  Keypad Row 4\nPA10 Keypad Col 1 + EEPROM_SCL (opt: SPI0 CLK)\nPA11 Keypad Col 2 + EEPROM_SDA (opt: SPI0 MISO)\nPA12 Keypad Col 3 + VOICE_0 (opt: SPI0 MOSI)\nPA13 Keypad Col 4 + VOICE_1"
     (at 370.078 452.12 0)
     (effects (font (size 1.27 1.27)) (justify left bottom))
   )
+  (text "VHF TX" (at 439.42 247.65 0)
+    (effects (font (size 1.27 1.27) (thickness 0.254) bold) (justify left bottom))
+  )
   (text "Keypad backlight" (at 617.982 368.554 0)
     (effects (font (size 1.27 1.27) (thickness 0.254) bold) (justify left bottom))
   )
+  (text "DC Path for TX UHF PIN" (at 669.29 243.84 0)
+    (effects (font (size 1.27 1.27) (thickness 0.254) bold) (justify left bottom))
+  )
+  (text "TX driver bias" (at 215.9 93.98 0)
+    (effects (font (size 1.27 1.27) (thickness 0.254) bold) (justify left bottom))
+  )

Commit message: Cleanup and additional notes
Cleanup of BK transceiver chip GPIO labels due to shared functions on TX and RX for band select
Some additional notes.
Other:
- note added: "31 nH?"
- note added: "Analog Bias for TX setpoints"
- note added: "BAND_UHF_EN"
- note added: "BAND_VHF_EN"
- note added: "Charge control based on VIN switching GND"
- note added: "Current sense node for TX final"
- note added: "Filtered RX to chip"
- note added: "Final gate bias network"
- note added: "LC microstrip filter?"
- note added: "Matching Cap Array on serpentine"
- note added: "Missing CC 5.1k resistors"
- note added: "Place one near TX, one near LNA transistors"
- note added: "SPARE_TP"
- note added: "Switched FM LNA"
- note added: "TX Power Bias"
- note added: "TX bias, initial filter"
- note added: "TX current sense for bias control"
- note added: "TX driver bias, filtered"
- note added: "UHF RX bias (PIN and LNA)"
- note added: "UHF pre-driver bias"
- note added: "VHF RX bias (PIN and LNA)"
- note added: "VHF TX PIN diode bias"
- note added: "VHF all 3 TX PIN diodes biased through LPF"
- note added: "VHF inductor, PIN out during UHF TX"
- note added: "VHF pre-driver bias"
- note removed: "RX_UHF_EN"
- note removed: "RX_VHF_EN"
- note removed: "TX driver bias"
- note removed: "TX_UHF_EN"
- note removed: "TX_VHF_EN"
Changed lines of the file:
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@@
     (comment 1 "Review, tidying: ludwich66 (GitHub)")
     (comment 2 "Reversing: MentalDetector (GitHub) / @philmcallen (Telegram)")
+    (comment 3 "RF Annotation: thomasrussellmurphy (GitHub)")
   )
   (junction (at 202.438 176.784) (diameter 0) (color 0 0 0 0)
@@
     (effects (font (size 1.27 1.27) (thickness 0.254) bold) (justify left bottom))
   )
-  (text "RX mute PIN" (at 650.24 129.54 0)
+  (text "VHF RX bias (PIN and LNA)" (at 473.71 49.53 0)
+    (effects (font (size 1.27 1.27) (thickness 0.254) bold) (justify left bottom))
+  )
+  (text "RX mute PIN" (at 650.24 134.62 0)
+    (effects (font (size 1.27 1.27) (thickness 0.254) bold) (justify left bottom))
+  )
+  (text "Charge control based on VIN switching GND" (at 627.38 541.02 0)
     (effects (font (size 1.27 1.27) (thickness 0.254) bold) (justify left bottom))
   )
@@
     (effects (font (size 1.27 1.27) (thickness 0.254) bold) (justify left bottom))
   )
+  (text "Switched FM LNA" (at 59.69 482.6 0)
+    (effects (font (size 1.27 1.27) (thickness 0.254) bold) (justify left bottom))
+  )
+  (text "Matching Cap Array on serpentine" (at 455.93 175.26 0)
+    (effects (font (size 1.27 1.27) (thickness 0.254) bold) (justify left bottom))
+  )
   (text "UHF LNA" (at 626.11 106.68 0)
     (effects (font (size 1.27 1.27) (thickness 0.254) bold) (justify left bottom))
@@
     (effects (font (size 1.27 1.27) (thickness 0.254) bold) (justify left bottom))
   )
+  (text "VHF pre-driver bias" (at 238.76 255.27 0)
+    (effects (font (size 1.27 1.27) (thickness 0.254) bold) (justify left bottom))
+  )
   (text "Regulated UHF PIN TX Bias?" (at 617.22 222.25 0)
     (effects (font (size 1.27 1.27) (thickness 0.254) bold) (justify left bottom))
@@
     (effects (font (size 1.27 1.27) (thickness 0.254) bold) (justify left bottom))
   )
+  (text "VHF TX PIN diode bias" (at 377.19 273.05 0)
+    (effects (font (size 1.27 1.27) (thickness 0.254) bold) (justify left bottom))
+  )
+  (text "Current sense node for TX final" (at 462.28 519.43 0)
+    (effects (font (size 1.27 1.27) (thickness 0.254) bold) (justify left bottom))
+  )
+  (text "VHF inductor, PIN out during UHF TX" (at 298.45 158.75 0)
+    (effects (font (size 1.27 1.27) (thickness 0.254) bold) (justify left bottom))
+  )
   (text "Combined volume pot.\n& ON/OFF Switch\n" (at 244.856 401.066 0)
     (effects (font (size 1.27 1.27) (thickness 0.254) bold) (justify left bottom))
   )
+  (text "SPARE_TP" (at 36.83 215.9 0)
+    (effects (font (size 1.27 1.27) (thickness 0.254) bold) (justify left bottom))
+  )
   (text "Half-duplex TDD FM Transceiver" (at 55.372 191.77 0)
     (effects (font (size 1.27 1.27) (thickness 0.254) bold) (justify left bottom))
   )
-  (text "RF driver" (at 231.648 144.526 0)
+  (text "RF driver" (at 224.79 191.77 0)
     (effects (font (size 1.27 1.27) (thickness 0.254) bold) (justify left bottom))
   )
@@
     (effects (font (size 1.27 1.27) (thickness 0.254) bold) (justify left bottom))
   )
+  (text "BAND_VHF_EN" (at 36.83 210.82 0)
+    (effects (font (size 1.27 1.27) (thickness 0.254) bold) (justify left bottom))
+  )
   (text "Charge LED" (at 461.518 350.012 0)
     (effects (font (size 1.27 1.27) (thickness 0.254) bold) (justify left bottom))
@@
     (effects (font (size 1.27 1.27)) (justify left bottom))
   )
+  (text "Place one near TX, one near LNA transistors" (at 650.24 137.16 0)
+    (effects (font (size 1.27 1.27) (thickness 0.254) bold) (justify left bottom))
+  )
+  (text "Analog Bias for TX setpoints" (at 74.93 85.09 0)
+    (effects (font (size 1.27 1.27) (thickness 0.254) bold) (justify left bottom))
+  )
+  (text "BAND_UHF_EN" (at 36.83 213.36 0)
+    (effects (font (size 1.27 1.27) (thickness 0.254) bold) (justify left bottom))
+  )
   (text "VHF/FM/Air pre-filter" (at 675.64 116.84 0)
     (effects (font (size 1.27 1.27) (thickness 0.254) bold) (justify left bottom))
@@
     (effects (font (size 1.27 1.27)) (justify left bottom))
   )
+  (text "UHF pre-driver bias" (at 233.68 210.82 0)
+    (effects (font (size 1.27 1.27) (thickness 0.254) bold) (justify left bottom))
+  )
   (text "Daughterboard\n" (at 270.51 393.954 0)
     (effects (font (size 1.27 1.27) (thickness 0.254) bold) (justify left bottom))
@@
     (effects (font (size 1.27 1.27) (thickness 0.254) bold) (justify left bottom))
   )
+  (text "TX Power Bias" (at 320.04 129.54 0)
+    (effects (font (size 1.27 1.27) (thickness 0.254) bold) (justify left bottom))
+  )
+  (text "TX Power Bias" (at 275.59 271.78 0)
+    (effects (font (size 1.27 1.27) (thickness 0.254) bold) (justify left bottom))
+  )
   (text "RX_EN" (at 411.48 130.81 0)
     (effects (font (size 1.27 1.27) (thickness 0.254) bold) (justify left bottom))
   )
-  (text "RX_VHF_EN" (at 414.02 59.69 0)
+  (text "BAND_VHF_EN" (at 414.02 59.69 0)
+    (effects (font (size 1.27 1.27) (thickness 0.254) bold) (justify left bottom))
+  )
+  (text "VHF all 3 TX PIN diodes biased through LPF" (at 662.94 267.97 0)
     (effects (font (size 1.27 1.27) (thickness 0.254) bold) (justify left bottom))
   )
@@
     (effects (font (size 1.27 1.27) (thickness 0.254) bold) (justify left bottom))
   )
-  (text "TX_VHF_EN" (at 267.97 292.1 0)
+  (text "BAND_VHF_EN" (at 267.97 292.1 0)
+    (effects (font (size 1.27 1.27) (thickness 0.254) bold) (justify left bottom))
+  )
+  (text "Final gate bias network" (at 374.65 200.66 0)
+    (effects (font (size 1.27 1.27) (thickness 0.254) bold) (justify left bottom))
+  )
+  (text "UHF RX bias (PIN and LNA)" (at 471.17 91.44 0)
     (effects (font (size 1.27 1.27) (thickness 0.254) bold) (justify left bottom))
   )
@@
     (effects (font (size 1.27 1.27) (thickness 0.254) bold) (justify left bottom))
   )
+  (text "TX bias, initial filter" (at 177.8 81.28 0)
+    (effects (font (size 1.27 1.27) (thickness 0.254) bold) (justify left bottom))
+  )
   (text "Battery filtering and current limiting" (at 396.748 520.954 0)
     (effects (font (size 1.27 1.27) (thickness 0.254) bold) (justify left bottom))
   )
-  (text "RX_UHF_EN" (at 406.4 101.6 0)
+  (text "TX_EN" (at 36.83 218.44 0)
+    (effects (font (size 1.27 1.27) (thickness 0.254) bold) (justify left bottom))
+  )
+  (text "BAND_UHF_EN" (at 406.4 101.6 0)
     (effects (font (size 1.27 1.27) (thickness 0.254) bold) (justify left bottom))
   )
@@
     (effects (font (size 1.27 1.27) (thickness 0.254) bold) (justify left bottom))
   )
+  (text "31 nH?" (at 274.32 160.02 0)
+    (effects (font (size 1.27 1.27) (thickness 0.254) bold) (justify left bottom))
+  )
+  (text "RX_EN" (at 36.83 220.98 0)
+    (effects (font (size 1.27 1.27) (thickness 0.254) bold) (justify left bottom))
+  )
   (text "RX LED" (at 498.856 350.012 0)
     (effects (font (size 1.27 1.27) (thickness 0.254) bold) (justify left bottom))
   )
-  (text "TX_UHF_EN" (at 267.97 243.84 0)
+  (text "TX Power Bias" (at 275.59 223.52 0)
+    (effects (font (size 1.27 1.27) (thickness 0.254) bold) (justify left bottom))
+  )
+  (text "BAND_UHF_EN" (at 267.97 243.84 0)
     (effects (font (size 1.27 1.27) (thickness 0.254) bold) (justify left bottom))
   )
@@
     (effects (font (size 1.27 1.27) (thickness 0.254) bold) (justify left bottom))
   )
+  (text "Missing CC 5.1k resistors" (at 534.67 488.95 0)
+    (effects (font (size 1.27 1.27) (thickness 0.254) bold) (justify left bottom))
+  )
+  (text "TX Power Bias" (at 715.01 124.46 0)
+    (effects (font (size 1.27 1.27) (thickness 0.254) bold) (justify left bottom))
+  )
   (text "Keypad backlight" (at 617.982 368.554 0)
     (effects (font (size 1.27 1.27) (thickness 0.254) bold) (justify left bottom))
   )
+  (text "TX current sense for bias control" (at 76.2 135.89 0)
+    (effects (font (size 1.27 1.27) (thickness 0.254) bold) (justify left bottom))
+  )
   (text "DC Path for TX UHF PIN" (at 669.29 243.84 0)
     (effects (font (size 1.27 1.27) (thickness 0.254) bold) (justify left bottom))
   )
-  (text "TX driver bias" (at 215.9 93.98 0)
+  (text "LC microstrip filter?" (at 455.93 177.8 0)
+    (effects (font (size 1.27 1.27) (thickness 0.254) bold) (justify left bottom))
+  )
+  (text "TX driver bias, filtered" (at 215.9 93.98 0)
     (effects (font (size 1.27 1.27) (thickness 0.254) bold) (justify left bottom))
   )
@@
     (effects (font (size 1.27 1.27)) (justify left bottom))
   )
+  (text "Filtered RX to chip" (at 524.51 78.74 0)
+    (effects (font (size 1.27 1.27) (thickness 0.254) bold) (justify left bottom))
+  )
   (global_label "DISP_6" (shape input) (at 712.47 503.174 180) (fields_autoplaced)
